Commit message: add housing

File: omo_r1mini_description/urdf/common_properties.xacro (robot description, xacro)
@@ -29,4 +29,7 @@
     <color rgba="0.8 0.0 0.0 1.0"/>
   </material>
+  <material name="pink">
+    <color rgba="${255/255} ${20/255} ${147/255} 1.0"/>
+  </material>
   <material name="white">
     <color rgba="1.0 1.0 1.0 1.0"/>

File: omo_r1mini_description/urdf/r1mini.urdf.xacro (robot description, xacro)
@@ -28,4 +28,31 @@
                iyy="8.6195418e-03" iyz="-3.5422299e-06"
                izz="1.4612727e-02" />
+    </inertial>
+  </link>
+  <joint name="housing_joint" type="fixed">
+    <parent link="base_link"/>
+    <child link="housing_link" />
+    <origin xyz="0 0 0" rpy="0 0 0.0"/>
+  </joint>
+  <link name="housing_link">
+    <visual>
+      <origin xyz="-0.028 0 -0.028" rpy="0 0 1.57"/>
+      <geometry>
+        <mesh filename="package://omo_r1mini_description/meshes/bases/mini_housing.stl" scale="0.001 0.001 0.001"/>
+      </geometry>
+      <material name="pink"/>
+    </visual>
+    <collision>
+      <origin xyz="-0.028 0 -0.028" rpy="0 0 1.57"/>
+      <geometry>
+        <mesh filename="package://omo_r1mini_description/meshes/bases/mini_housing.stl" scale="0.001 0.001 0.001"/>
+      </geometry>
+    </collision>
+    <inertial>
+      <origin xyz="-0.1 0 0" rpy="0 0 0"/>
+      <mass value="0.01"/>
+      <inertia ixx="8.7002718e-04" ixy="-4.7576583e-07" ixz="1.1160499e-07"
+               iyy="8.6195418e-04" iyz="-3.5422299e-07"
+               izz="1.4612727e-04" />
     </inertial>
   </link>
@@ -122,5 +149,5 @@
     <parent link="base_link"/>
     <child link="base_scan"/>
-    <origin xyz="0.0 0 0.05" rpy="0.0 0 3.14159"/>
+    <origin xyz="0.0 0 0.07" rpy="0.0 0 3.14159"/>
   </joint>
   <link name="base_scan">

File: omo_r1mini_gazebo/sdf/omo_r1mini.gazebo.xacro (robot description, xacro)
@@ -13,4 +13,7 @@
   <gazebo reference="wheel_right_link">
     <material>Gazebo/FlatBlack</material>
+  </gazebo>
+  <gazebo reference="housing_link">
+    <material>Gazebo/PurpleGlow</material>
   </gazebo>
   <gazebo reference="caster_back_link">
