Commit message: bug fix

File: omo_r1mini_description/urdf/r1mini.urdf.hlds.xacro (robot description, xacro)
@@ -149,5 +149,5 @@
     <parent link="base_link"/>
     <child link="base_scan"/>
-    <origin xyz="0.0 0 0.07" rpy="0.0 0.01667 3.14159"/>
+    <origin xyz="0.0 0 0.07" rpy="0.0 -0.01667 3.14159"/>
   </joint>
   <link name="base_scan">

Commit message: bug fix

File: omo_r1mini_description/urdf/r1mini.urdf.hlds.xacro (robot description, xacro)
@@ -149,5 +149,5 @@
     <parent link="base_link"/>
     <child link="base_scan"/>
-    <origin xyz="0.0 0 0.07" rpy="0.0 -0.01667 3.14159"/>
+    <origin xyz="-0.005 0 0.07" rpy="0.0 -0.01667 3.14159"/>
   </joint>
   <link name="base_scan">

Commit message: bug fix

File: omo_r1mini_description/urdf/r1mini.urdf.hlds.xacro (robot description, xacro)
@@ -6,5 +6,5 @@
     <parent link="base_footprint"/>
     <child link="base_link" />
-    <origin xyz="0 0 0.0335" rpy="0 0 0.0"/>
+    <origin xyz="0 0 0.0335" rpy="0 -0.01667 0.0"/>
   </joint>
   <link name="base_link">
@@ -149,5 +149,5 @@
     <parent link="base_link"/>
     <child link="base_scan"/>
-    <origin xyz="-0.005 0 0.07" rpy="0.0 -0.01667 3.14159"/>
+    <origin xyz="-0.005 0 0.07" rpy="0.0 0.0 3.14159"/>
   </joint>
   <link name="base_scan">

Commit message: bug fix

File: omo_r1mini_description/urdf/r1mini.urdf.hlds.xacro (robot description, xacro)
@@ -6,5 +6,5 @@
     <parent link="base_footprint"/>
     <child link="base_link" />
-    <origin xyz="0 0 0.0335" rpy="0 -0.01667 0.0"/>
+    <origin xyz="0 0 0.0335" rpy="0 0.0 0.0"/>
   </joint>
   <link name="base_link">
@@ -149,5 +149,5 @@
     <parent link="base_link"/>
     <child link="base_scan"/>
-    <origin xyz="-0.005 0 0.07" rpy="0.0 0.0 3.14159"/>
+    <origin xyz="-0.002 0 0.07" rpy="0.0 0.02 3.14159"/>
   </joint>
   <link name="base_scan">

Commit message: bug fix

File: omo_r1mini_description/urdf/r1mini.urdf.hlds.xacro (robot description, xacro)
@@ -149,5 +149,5 @@
     <parent link="base_link"/>
     <child link="base_scan"/>
-    <origin xyz="-0.002 0 0.07" rpy="0.0 0.02 3.14159"/>
+    <origin xyz="-0.002 0 0.07" rpy="0.0 0.034 3.14159"/>
   </joint>
   <link name="base_scan">
