Commit message: add gazebo pkg

File: omo_r1mini_description/urdf/r1mini.urdf.xacro (robot description, xacro)
@@ -114,3 +114,36 @@
     </inertial>
   </link>
+  <joint name="imu_joint" type="fixed">
+    <parent link="base_link"/>
+    <child link="imu_link"/>
+    <origin xyz="0.0 0 0.038" rpy="0 0 0"/>
+  </joint>
+  <link name="imu_link"/>
+  <joint name="scan_joint" type="fixed">
+    <parent link="base_link"/>
+    <child link="base_scan"/>
+    <origin xyz="0.0 0 0.13" rpy="0.0 0 3.14159"/>
+  </joint>
+  <link name="base_scan">
+    <visual>
+      <origin xyz="0 0 0.0" rpy="0 0 0"/>
+      <geometry>
+        <mesh filename="package://omo_r1mini_description/meshes/sensors/lds.stl" scale="0.001 0.001 0.001"/>
+      </geometry>
+      <material name="dark"/>
+    </visual>
+    <collision>
+      <origin xyz="0.015 0 -0.0065" rpy="0 0 0"/>
+      <geometry>
+        <cylinder length="0.0315" radius="0.055"/>
+      </geometry>
+    </collision>
+    <inertial>
+      <mass value="0.114" />
+      <origin xyz="0 0 0" />
+      <inertia ixx="0.001" ixy="0.0" ixz="0.0"
+               iyy="0.001" iyz="0.0"
+               izz="0.001" />
+    </inertial>
+  </link>
 </robot>

Commit message: bug fix on gazebo

File: omo_r1mini_description/urdf/r1mini.urdf.xacro (robot description, xacro)
@@ -1,15 +1,15 @@
 <?xml version="1.0" ?>
 <robot name="r1mini" xmlns:xacro="http://ros.org/wiki/xacro">
-  <xacro:include filename="$(find omo_r1mini_description)/urdf/common_properties.xacro"/>
-  <xacro:include filename="$(find omo_r1mini_description)/urdf/r1mini.gazebo.xacro"/>
+<!--   <xacro:include filename="$(find omo_r1mini_description)/urdf/common_properties.xacro"/>
+ -->
   <link name="base_footprint"/>
   <joint name="base_joint" type="fixed">
     <parent link="base_footprint"/>
     <child link="base_link" />
-    <origin xyz="0 0.0 0.0115" rpy="0 0 0.0"/>
+    <origin xyz="0 0 0.0335" rpy="0 0 0.0"/>
   </joint>
   <link name="base_link">
     <visual>
-      <origin xyz="0.03 -0.065 0.0" rpy="0 0 1.57"/>
+      <origin xyz="0.03 -0.065 -0.022" rpy="0 0 1.57"/>
       <geometry>
         <mesh filename="package://omo_r1mini_description/meshes/bases/mini_frame.stl" scale="0.001 0.001 0.001"/>
@@ -18,5 +18,5 @@
     </visual>
     <collision>
-      <origin xyz="0.03 -0.065 0.0" rpy="0 0 1.57"/>
+      <origin xyz="0.03 -0.065 -0.022" rpy="0 0 1.57"/>
       <geometry>
         <mesh filename="package://omo_r1mini_description/meshes/bases/mini_frame.stl" scale="0.001 0.001 0.001"/>
@@ -34,5 +34,5 @@
     <parent link="base_link"/>
     <child link="wheel_left_link"/>
-    <origin xyz="0.0 0.096 0.022" rpy="0.0 0.0 0"/>
+    <origin xyz="0.0 0.096 0.0" rpy="0.0 0.0 0"/>
     <axis xyz="0 1 0"/>
   </joint>
@@ -62,5 +62,5 @@
     <parent link="base_link"/>
     <child link="wheel_right_link"/>
-    <origin xyz="0.0 -0.096 0.022" rpy="0.0 0.0 0"/>
+    <origin xyz="0.0 -0.096 0.0" rpy="0.0 0.0 0"/>
     <axis xyz="0 1 0"/>
   </joint>
@@ -90,5 +90,5 @@
     <parent link="base_link"/>
     <child link="caster_back_link"/>
-    <origin xyz="-0.12 0.0 0.0" rpy="0 0 0"/>
+    <origin xyz="-0.12 0.0 -0.022" rpy="0 0 0"/>
   </joint>
   <link name="caster_back_link">

File: omo_r1mini_gazebo/sdf/omo_r1mini.gazebo.xacro (robot description, xacro)
@@ -54,5 +54,5 @@
   </gazebo>
   <gazebo>
-    <plugin name="omo_r1_controller" filename="libgazebo_ros_diff_drive.so">
+    <plugin name="omo_r1mini_controller" filename="libgazebo_ros_diff_drive.so">
       <commandTopic>cmd_vel</commandTopic>
       <odometryTopic>odom</odometryTopic>
@@ -68,6 +68,6 @@
       <leftJoint>wheel_left_joint</leftJoint>
       <rightJoint>wheel_right_joint</rightJoint>
-      <wheelSeparation>0.591</wheelSeparation>
-      <wheelDiameter>0.220</wheelDiameter>
+      <wheelSeparation>0.17</wheelSeparation>
+      <wheelDiameter>0.0675</wheelDiameter>
       <wheelAcceleration>1</wheelAcceleration>
       <wheelTorque>100</wheelTorque>

Commit message: bug

File: omo_r1mini_description/urdf/r1mini.urdf.xacro (robot description, xacro)
@@ -1,6 +1,5 @@
 <?xml version="1.0" ?>
 <robot name="r1mini" xmlns:xacro="http://ros.org/wiki/xacro">
-<!--   <xacro:include filename="$(find omo_r1mini_description)/urdf/common_properties.xacro"/>
- -->
+  <xacro:include filename="$(find omo_r1mini_description)/urdf/common_properties.xacro"/>
   <link name="base_footprint"/>
   <joint name="base_joint" type="fixed">
@@ -24,5 +23,5 @@
     </collision>
     <inertial>
-      <origin xyz="0 0 0" rpy="0 0 0"/>
+      <origin xyz="0 -0.1 0" rpy="0 0 0"/>
       <mass value="1.3729096e+00"/>
       <inertia ixx="8.7002718e-03" ixy="-4.7576583e-05" ixz="1.1160499e-04"
@@ -90,5 +89,5 @@
     <parent link="base_link"/>
     <child link="caster_back_link"/>
-    <origin xyz="-0.12 0.0 -0.022" rpy="0 0 0"/>
+    <origin xyz="-0.12 0.0 -0.018" rpy="0 0 0"/>
   </joint>
   <link name="caster_back_link">
@@ -123,5 +122,5 @@
     <parent link="base_link"/>
     <child link="base_scan"/>
-    <origin xyz="0.0 0 0.13" rpy="0.0 0 3.14159"/>
+    <origin xyz="0.0 0 0.05" rpy="0.0 0 3.14159"/>
   </joint>
   <link name="base_scan">
@@ -140,5 +139,5 @@
     </collision>
     <inertial>
-      <mass value="0.114" />
+      <mass value="0.05" />
       <origin xyz="0 0 0" />
       <inertia ixx="0.001" ixy="0.0" ixz="0.0"

Commit message: fix bug in gazebo

File: omo_r1mini_description/urdf/r1mini.urdf.xacro (robot description, xacro)
@@ -23,5 +23,5 @@
     </collision>
     <inertial>
-      <origin xyz="0 -0.1 0" rpy="0 0 0"/>
+      <origin xyz="-0.1 0 0" rpy="0 0 0"/>
       <mass value="1.3729096e+00"/>
       <inertia ixx="8.7002718e-03" ixy="-4.7576583e-05" ixz="1.1160499e-04"

File: omo_r1mini_gazebo/sdf/omo_r1mini.gazebo.xacro (robot description, xacro)
@@ -2,46 +2,19 @@
 <robot name="omo_r1_sim" xmlns:xacro="http://ros.org/wiki/xacro">
   <xacro:include filename="$(find omo_r1mini_description)/urdf/r1mini.urdf.xacro"/>
-  <xacro:arg name="laser_visual"  default="false"/>
+  <xacro:arg name="laser_visual"  default="true"/>
   <xacro:arg name="camera_visual" default="false"/>
-  <xacro:arg name="imu_visual"    default="false"/>
+  <xacro:arg name="imu_visual"    default="true"/>
   <gazebo reference="base_link">
     <material>Gazebo/DarkGrey</material>
   </gazebo>
   <gazebo reference="wheel_left_link">
-    <mu1>1.0</mu1>
-    <mu2>1.0</mu2>
-    <kp>50000.0</kp>
-    <kd>1.0</kd>
-    <minDepth>0.001</minDepth>
-    <maxVel>1.2</maxVel>
-    <fdir1>1 0 0</fdir1>
     <material>Gazebo/FlatBlack</material>
   </gazebo>
   <gazebo reference="wheel_right_link">
-    <mu1>1.0</mu1>
-    <mu2>1.0</mu2>
-    <kp>50000.0</kp>
-    <kd>1.0</kd>
-    <minDepth>0.001</minDepth>
-    <maxVel>1.2</maxVel>
-    <fdir1>1 0 0</fdir1>
     <material>Gazebo/FlatBlack</material>
   </gazebo>
-  <gazebo reference="caster_back_right_link">
-    <mu1>0.1</mu1>
-    <mu2>0.1</mu2>
-    <kp>10000.0</kp>
-    <kd>10.0</kd>
-    <minDepth>0.001</minDepth>
-    <maxVel>1.0</maxVel>
-    <material>Gazebo/FlatBlack</material>
-  </gazebo>
-  <gazebo reference="caster_back_left_link">
-    <mu1>0.1</mu1>
-    <mu2>0.1</mu2>
-    <kp>10000.0</kp>
-    <kd>10.0</kd>
-    <minDepth>0.001</minDepth>
-    <maxVel>1.0</maxVel>
+  <gazebo reference="caster_back_link">
+    <mu1>0</mu1>
+    <mu2>0</mu2>
     <material>Gazebo/FlatBlack</material>
   </gazebo>

Commit message: add housing

File: omo_r1mini_description/urdf/r1mini.urdf.xacro (robot description, xacro)
@@ -14,5 +14,5 @@
         <mesh filename="package://omo_r1mini_description/meshes/bases/mini_frame.stl" scale="0.001 0.001 0.001"/>
       </geometry>
-      <material name="blue"/>
+      <material name="dark"/>
     </visual>
     <collision>

File: omo_r1mini_gazebo/sdf/omo_r1mini.gazebo.xacro (robot description, xacro)
@@ -2,9 +2,9 @@
 <robot name="omo_r1_sim" xmlns:xacro="http://ros.org/wiki/xacro">
   <xacro:include filename="$(find omo_r1mini_description)/urdf/r1mini.urdf.xacro"/>
-  <xacro:arg name="laser_visual"  default="true"/>
+  <xacro:arg name="laser_visual"  default="false"/>
   <xacro:arg name="camera_visual" default="false"/>
   <xacro:arg name="imu_visual"    default="true"/>
   <gazebo reference="base_link">
-    <material>Gazebo/DarkGrey</material>
+    <material>Gazebo/Indigo</material>
   </gazebo>
   <gazebo reference="wheel_left_link">

Commit message: add hlds

File: omo_r1mini_description/urdf/r1mini.urdf.xacro (robot description, xacro)
@@ -39,5 +39,5 @@
       <origin xyz="-0.028 0 -0.028" rpy="0 0 1.57"/>
       <geometry>
-        <mesh filename="package://omo_r1mini_description/meshes/bases/mini_housing.stl" scale="0.001 0.001 0.001"/>
+        <mesh filename="package://omo_r1mini_description/meshes/bases/mini_housing lite 2.stl" scale="0.001 0.001 0.001"/>
       </geometry>
       <material name="pink"/>

Commit message: bug fix

File: omo_r1mini_description/urdf/r1mini.urdf.xacro (robot description, xacro)
@@ -39,5 +39,5 @@
       <origin xyz="-0.028 0 -0.028" rpy="0 0 1.57"/>
       <geometry>
-        <mesh filename="package://omo_r1mini_description/meshes/bases/mini_housing lite 2.stl" scale="0.001 0.001 0.001"/>
+        <mesh filename="package://omo_r1mini_description/meshes/bases/r1mini housing lite 2.stl" scale="0.001 0.001 0.001"/>
       </geometry>
       <material name="pink"/>
@@ -46,5 +46,5 @@
       <origin xyz="-0.028 0 -0.028" rpy="0 0 1.57"/>
       <geometry>
-        <mesh filename="package://omo_r1mini_description/meshes/bases/mini_housing.stl" scale="0.001 0.001 0.001"/>
+        <mesh filename="package://omo_r1mini_description/meshes/bases/r1mini housing lite 2.stl" scale="0.001 0.001 0.001"/>
       </geometry>
     </collision>

Commit message: add ar marker

File: omo_r1mini_description/urdf/r1mini.urdf.xacro (robot description, xacro)
@@ -173,3 +173,9 @@
     </inertial>
   </link>
+  <joint name="camera_joint" type="fixed">
+    <origin xyz="0.02 0 0.02" rpy="0 0 0"/>
+    <parent link="base_link"/>
+    <child link="camera_frame"/>
+  </joint>
+  <link name="camera_frame"/>
 </robot>

Commit message: Update r1mini.urdf.xacro

File: omo_r1mini_description/urdf/r1mini.urdf.xacro (robot description, xacro)
@@ -174,5 +174,5 @@
   </link>
   <joint name="camera_joint" type="fixed">
-    <origin xyz="0.02 0 0.02" rpy="0 0 0"/>
+    <origin xyz="0.04 0 0.02" rpy="0 0 0"/>
     <parent link="base_link"/>
     <child link="camera_frame"/>

Commit message: Update r1mini.urdf.xacro

File: omo_r1mini_description/urdf/r1mini.urdf.xacro (robot description, xacro)
@@ -178,4 +178,4 @@
     <child link="camera_frame"/>
   </joint>
-  <link name="camera_frame"/>
+  <link name="main_camera_optical"/>
 </robot>

Commit message: Update r1mini.urdf.xacro

File: omo_r1mini_description/urdf/r1mini.urdf.xacro (robot description, xacro)
@@ -176,5 +176,5 @@
     <origin xyz="0.04 0 0.02" rpy="0 0 0"/>
     <parent link="base_link"/>
-    <child link="camera_frame"/>
+    <child link="main_camera_optical"/>
   </joint>
   <link name="main_camera_optical"/>

Commit message: minor change

File: omo_r1mini_description/urdf/r1mini.urdf.xacro (robot description, xacro)
@@ -174,5 +174,5 @@
   </link>
   <joint name="camera_joint" type="fixed">
-    <origin xyz="0.04 0 0.02" rpy="0 0 0"/>
+    <origin xyz="0.04 0 0.02" rpy="0 1.570796 0"/>
     <parent link="base_link"/>
     <child link="main_camera_optical"/>

Commit message: changes

File: omo_r1mini_description/urdf/r1mini.urdf.xacro (robot description, xacro)
@@ -174,5 +174,5 @@
   </link>
   <joint name="camera_joint" type="fixed">
-    <origin xyz="0.04 0 0.02" rpy="0 1.570796 0"/>
+    <origin xyz="0.04 0 0.02" rpy="3.14159 -1.570796 0"/>
     <parent link="base_link"/>
     <child link="main_camera_optical"/>
