Commit message: bug fix

File: omo_r1mini_description/urdf/r1mini_upcamera.urdf.xacro (robot description, xacro)
@@ -174,5 +174,5 @@
   </link>
   <joint name="camera_joint" type="fixed">
-    <origin xyz="0.06 0 0.06" rpy="0 0 0"/>
+    <origin xyz="0.06 0 0.06" rpy="0 0 1.570796"/>
     <parent link="base_link"/>
     <child link="main_camera_optical"/>
